Commit message: gazebo complete

File: kwj_description/urdf/kwj.urdf.xacro (robot description, xacro)
@@ -10,7 +10,7 @@
   <link name="base_link">
     <inertial>
-      <origin xyz="0.155 0.2 0.2"/>
+      <origin xyz="0 0 0" rpy="0 0 0"/>
       <mass value="1.0" />
-      <inertia ixx="0.1" ixy="0" ixz="0" iyy="0.1" iyz="0" izz="0.1" />
+      <inertia ixx="8.7002718e-03" ixy="-4.7576583e-05" ixz="1.1160499e-04" iyy="8.6195418e-03" iyz="-3.5422299e-06" izz="1.4612727e-02" />
     </inertial>
     <collision>
